Commit message: add tcp link

File: descriptions/pisoftgrip_description/urdf/pisoftgrip_macro.xacro (robot description, xacro)
@@ -22,4 +22,11 @@
         </collision>
     </link>
+    <joint name="${prefix}pisoftgrip_tcp_joint" type="fixed">
+        <parent link="${prefix}pisoftgrip_link"/>
+        <child link="${prefix}pisoftgrip_tcp"/>
+        <origin xyz="0 0 -0.06" rpy="0 0 0"/>
+    </joint>
+    <link name="${prefix}pisoftgrip_tcp">
+    </link>
     </xacro:macro>
 </robot>
