Commit message: added realsense urdf

File: descriptions/workcell_description/urdf/workcell.urdf.xacro (robot description, xacro)
@@ -4,7 +4,11 @@
   <xacro:arg name="ur_type" default="ur5e"/>
   <xacro:arg name="joint_limits_parameters_file" default="$(find ur_description)/config/$(arg ur_type)/joint_limits.yaml"/>
-  <xacro:arg name="kinematics_parameters_file" default="$(find ur_description)/config/$(arg ur_type)/default_kinematics.yaml"/>
+  <xacro:arg name="kinematics_parameters_file" default="$(find workcell_description)/config/my_robot_calibration.yaml"/>
   <xacro:arg name="physical_parameters_file" default="$(find ur_description)/config/$(arg ur_type)/physical_parameters.yaml"/>
   <xacro:arg name="visual_parameters_file" default="$(find ur_description)/config/$(arg ur_type)/visual_parameters.yaml"/>
+  <!-- Arguments for the Realsense D415 -->
+  <xacro:arg name="use_nominal_extrinsics" default="false" />
+  <xacro:arg name="add_plug" default="true" />
+  <xacro:arg name="use_mesh" default="false" />
   <!-- World Link (represents the origin of the world coordinate frame) -->
   <link name="world"/>
@@ -17,6 +21,9 @@
     physical_parameters_file="$(arg physical_parameters_file)"
     visual_parameters_file="$(arg visual_parameters_file)"
+    use_nominal_extrinsics="$(arg use_nominal_extrinsics)"
+    add_plug="$(arg add_plug)"
+    use_mesh="$(arg use_mesh)"
     >
-    <origin xyz="0 0 1" rpy="0 0 0" />
+    <origin xyz="0 0 0" rpy="0 0 0" />
   </xacro:workcell>
 </robot>

File: descriptions/workcell_description/urdf/workcell_macro.xacro (robot description, xacro)
@@ -5,4 +5,5 @@
   <xacro:include filename="$(find pisoftgrip_description)/urdf/pisoftgrip_macro.xacro"/>
   <xacro:include filename="$(find environment_description)/urdf/environment_macro.xacro"/>
+  <xacro:include filename="$(find realsense2_description)/urdf/_d415.urdf.xacro"/>
   <xacro:macro name="workcell" params="
     parent
@@ -13,4 +14,7 @@
     physical_parameters_file
     visual_parameters_file
+    use_nominal_extrinsics
+    add_plug
+    use_mesh
     ">
     <!-- Environment -->
@@ -46,4 +50,13 @@
     <!-- Piab PiSoftGripper -->
     <xacro:pisoftgrip prefix=""/>
+    <!-- Realsense D415 -->
+    <xacro:sensor_d415
+        name="d415"
+        parent="robot_mount"
+        use_nominal_extrinsics="${use_nominal_extrinsics}"
+        add_plug="${add_plug}"
+        use_mesh="${use_mesh}">
+      <origin xyz="0.3 0 0.15" rpy="0 0 0"/>
+    </xacro:sensor_d415>
   </xacro:macro>
 </robot>
