Commit message: update urdf: rotate base

File: descriptions/workcell_description/urdf/workcell_macro.xacro (robot description, xacro)
@@ -31,5 +31,5 @@
       generate_ros2_control_tag="false"
       >
-      <origin xyz="0 0 0" rpy="0 0 0"/>
+      <origin xyz="0 0 0" rpy="0 0 -1.5708"/>
     </xacro:ur_robot>
     <!-- Robot (Tool0) to Robotiq Epick -->

Commit message: update camera position

File: descriptions/workcell_description/urdf/workcell_macro.xacro (robot description, xacro)
@@ -57,5 +57,5 @@
         add_plug="${add_plug}"
         use_mesh="${use_mesh}">
-      <origin xyz="0.30 0 0.11" rpy="0 0 0"/>
+      <origin xyz="0.25 0 0.11" rpy="0 0 0"/>
     </xacro:sensor_d415>
   </xacro:macro>

Commit message: added link d415_sim_optical_frame for webots realsense

File: descriptions/workcell_description/urdf/workcell_macro.xacro (robot description, xacro)
@@ -6,4 +6,5 @@
   <xacro:include filename="$(find environment_description)/urdf/environment_macro.xacro"/>
   <xacro:include filename="$(find realsense2_description)/urdf/_d415.urdf.xacro"/>
+  <xacro:property name="M_PI" value="3.1415926535897931"/>
   <xacro:macro name="workcell" params="
     parent
@@ -59,4 +60,13 @@
       <origin xyz="0.25 0 0.11" rpy="0 0 0"/>
     </xacro:sensor_d415>
+    <!-- ===== Simulations-Frame am PROTO-Zentrum ===== -->
+    <link name="d415_sim_optical_frame"/>
+    <joint name="d415_sim_optical_joint" type="fixed">
+      <parent link="d415_bottom_screw_frame"/>
+      <child link="d415_sim_optical_frame"/>
+      <!-- XY = 0: mittig wie bottom_screw
+          Z = halbe Gehäusehöhe (0.023/2 = 0.0115): Sensormitte -->
+      <origin xyz="0 0 0.0115" rpy="${-M_PI/2} 0 ${-M_PI/2}"/>
+    </joint>
   </xacro:macro>
 </robot>

Commit message: fix(workcell_macro.xacro): adjust D415 sensor origin height for improved alignment

File: descriptions/workcell_description/urdf/workcell_macro.xacro (robot description, xacro)
@@ -57,5 +57,5 @@
         add_plug="${add_plug}"
         use_mesh="${use_mesh}">
-      <origin xyz="0.25 0 0.11" rpy="0 0 0"/>
+      <origin xyz="0.25 0 0.115" rpy="0 0 0"/>
     </xacro:sensor_d415>
     <!-- ===== Simulations-Frame am PROTO-Zentrum ===== -->
