Commit message: update descriptions

File: descriptions/epick_gripper_description/urdf/epick_macro_with_end_effector.xacro (robot description, xacro)
@@ -49,10 +49,10 @@
       <parent link="${hand_link_name}"/>
       <child link="epick_end_effector"/>
-      <origin xyz="0 0 ${0.13}" rpy="0 0 0"/>
+      <origin xyz="0 0 ${0.115}" rpy="0 0 0"/>
     </joint>
     <link name="epick_end_effector">
       <gravity>0</gravity>
       <visual>
-        <origin rpy="0 0 0.005" xyz="0 0 0"/>
+        <origin rpy="0 0 0" xyz="0 0 0"/>
         <geometry>
           <cylinder radius="0.0225" length="0.01"/>

File: descriptions/epick_gripper_description/urdf/robotiq_epick_model_macro.xacro (robot description, xacro)
@@ -40,5 +40,5 @@
       <parent link="${hand_link_name}"/>
       <child link="epick_end_effector"/>
-      <origin xyz="0 0 0.12" rpy="0 0 0"/>
+      <origin xyz="0 0 0.115" rpy="0 0 0"/>
     </joint>
     <link name="epick_end_effector"/>

File: descriptions/pisoftgrip_description/urdf/pisoftgrip_macro.xacro (robot description, xacro)
@@ -2,4 +2,10 @@
 <robot xmlns:xacro="http://wiki.ros.org/xacro">
     <xacro:macro name="pisoftgrip" params="prefix">
+    <link name="${prefix}pisoftgrip_flansch"/>
+    <joint name="${prefix}pisoftgrip_link_to_flansch" type="fixed">
+        <parent link="${prefix}pisoftgrip_flansch"/>
+        <child link="${prefix}pisoftgrip_link"/>
+        <origin xyz="0 0 0.018" rpy="0 0 0"/>
+    </joint>
     <link name="${prefix}pisoftgrip_link">
         <inertial>
@@ -9,4 +15,5 @@
         </inertial>
         <visual>
+            <origin xyz="0 0 0" rpy="0 3.141592653589 0"/>
             <geometry>
                 <mesh filename="package://pisoftgrip_description/meshes/pisoftgrip.stl" />
@@ -17,4 +24,5 @@
         </visual>
         <collision>
+            <origin xyz="0 0 0" rpy="0 3.141592653589 0"/>
             <geometry>
                 <mesh filename="package://pisoftgrip_description/meshes/pisoftgrip_simplified_605_faces.stl" />
@@ -22,11 +30,10 @@
         </collision>
     </link>
+    <link name="${prefix}pisoftgrip_tcp"/>
     <joint name="${prefix}pisoftgrip_tcp_joint" type="fixed">
-        <parent link="${prefix}pisoftgrip_link"/>
+        <parent link="${prefix}pisoftgrip_flansch"/>
         <child link="${prefix}pisoftgrip_tcp"/>
-        <origin xyz="0 0 -0.06" rpy="0 0 0"/>
+        <origin xyz="0 0 0.08" rpy="0 0 0"/>
     </joint>
-    <link name="${prefix}pisoftgrip_tcp">
-    </link>
     </xacro:macro>
 </robot>

File: descriptions/workcell_description/urdf/workcell.urdf.xacro (robot description, xacro)
@@ -10,5 +10,5 @@
   <xacro:arg name="use_nominal_extrinsics" default="false" />
   <xacro:arg name="add_plug" default="true" />
-  <xacro:arg name="use_mesh" default="false" />
+  <xacro:arg name="use_mesh" default="true" />
   <!-- World Link (represents the origin of the world coordinate frame) -->
   <link name="world"/>

File: descriptions/workcell_description/urdf/workcell_macro.xacro (robot description, xacro)
@@ -45,6 +45,6 @@
     <joint name="epick_to_pisoftgrip" type="fixed">
       <parent link="epick_end_effector"/>
-      <child link="pisoftgrip_link"/>
-      <origin xyz="0 0 0" rpy="0 3.14159265359 0" />
+      <child link="pisoftgrip_flansch"/>
+      <origin xyz="0 0 0" rpy="0 0 0" />
     </joint>
     <!-- Piab PiSoftGripper -->
@@ -57,5 +57,5 @@
         add_plug="${add_plug}"
         use_mesh="${use_mesh}">
-      <origin xyz="0.3 0 0.15" rpy="0 0 0"/>
+      <origin xyz="0.30 0 0.11" rpy="0 0 0"/>
     </xacro:sensor_d415>
   </xacro:macro>
