Commit message: changed joint name

File: descriptions/environment_description/urdf/environment_macro.xacro (robot description, xacro)
@@ -15,6 +15,6 @@
     <xacro:property name="robot_mount_y" value="0.335"/>
     <!-- /Parameters -->
-    <!-- World to Table -->
-    <joint name="world_to_table" type="fixed">
+    <!-- Table to World -->
+    <joint name="table_to_world" type="fixed">
       <parent link="${parent}"/>
       <child link="table"/>

Commit message: update robot_mount_y value to table center

File: descriptions/environment_description/urdf/environment_macro.xacro (robot description, xacro)
@@ -13,5 +13,5 @@
     <!-- Robot Mount Parameters -->
     <xacro:property name="robot_mount_x" value="0.24"/>
-    <xacro:property name="robot_mount_y" value="0.335"/>
+    <xacro:property name="robot_mount_y" value="0.325"/>
     <!-- /Parameters -->
     <!-- Table to World -->
