Commit message: updated realsense proto and urdf, now working and publishing

File: workcell/workcell_webots/config/realsense_d415_webots.urdf.xacro (robot description, xacro)
@@ -3,4 +3,5 @@
   <!-- D415 macro aus dem offiziellen realsense2_description -->
   <xacro:include filename="$(find realsense2_description)/urdf/_d415.urdf.xacro"/>
+  <xacro:property name="M_PI" value="3.1415926535897931"/>
   <!-- Root -->
   <link name="world"/>
@@ -14,18 +15,32 @@
     <origin xyz="0 0 0" rpy="0 0 0"/>
   </xacro:sensor_d415>
+  <!-- ===== Simulations-Frame am PROTO-Zentrum ===== -->
+  <link name="d415_sim_optical_frame"/>
+  <joint name="d415_sim_optical_joint" type="fixed">
+    <parent link="d415_bottom_screw_frame"/>
+    <child link="d415_sim_optical_frame"/>
+    <!-- XY = 0: mittig wie bottom_screw
+         Z = halbe Gehäusehöhe (0.023/2 = 0.0115): Sensormitte -->
+    <origin xyz="0 0 0.0115" rpy="${-M_PI/2} 0 ${-M_PI/2}"/>
+  </joint>
   <!-- Webots device mapping -->
   <webots>
-    <device reference="realsense_rgb" type="Camera">
-      <ros>
-        <topicName>/camera/color/image_raw</topicName>
-        <alwaysOn>true</alwaysOn>
-      </ros>
-    </device>
-    <device reference="realsense_depth" type="RangeFinder">
-      <ros>
-        <topicName>/camera/depth/image_rect_raw</topicName>
-        <alwaysOn>true</alwaysOn>
-      </ros>
-    </device>
-  </webots>
+  <device reference="realsense_rgb" type="Camera">
+    <ros>
+      <topicName>/webots_realsense/color/image_raw</topicName>
+      <frameName>d415_sim_optical_frame</frameName>
+      <alwaysOn>true</alwaysOn>
+      <enabled>true</enabled>
+    </ros>
+  </device>
+  <device reference="realsense_depth" type="RangeFinder">
+    <ros>
+      <topicName>/webots_realsense/depth/image_rect_raw</topicName>
+      <!-- Same frame name as camera because real realsense uses align_depth:=true -->
+      <frameName>d415_sim_optical_frame</frameName>
+      <alwaysOn>true</alwaysOn>
+      <enabled>true</enabled>
+    </ros>
+  </device>
+</webots>
 </robot>

File: workcell/workcell_webots/config/ur5e_webots.urdf.xacro (robot description, xacro)
@@ -1,4 +1,5 @@
 <?xml version="1.0"?>
 <robot name="ur5e" xmlns:xacro="http://www.ros.org/wiki/xacro">
+    <!-- Args -->
     <xacro:arg name="initial_positions_file" default="initial_positions.yaml" />
     <xacro:arg name="ur_type" default="ur5e"/>
@@ -7,10 +8,16 @@
     <xacro:arg name="physical_parameters_file" default="$(find ur_description)/config/$(arg ur_type)/physical_parameters.yaml"/>
     <xacro:arg name="visual_parameters_file" default="$(find ur_description)/config/$(arg ur_type)/visual_parameters.yaml"/>
+    <!-- URDF macros for the UR5e -->
     <xacro:include filename="$(find ur_description)/urdf/ur_macro.xacro"/>
     <webots>
+        <!-- Ros2Control plugin for the UR5e -->
         <plugin type="webots_ros2_control::Ros2Control"/>
     </webots>
+    <!-- Include the ROS2 Control configuration for the UR5e -->
     <xacro:include filename="ur5e_webots.ros2_control.xacro" />
+    <xacro:workcell_ros2_control name="WebotsControl" initial_positions_file="$(arg initial_positions_file)"/>
+    <!-- Root link -->
     <link name="world"/>
+    <!-- UR5e Robot -->
     <xacro:ur_robot
         name="$(arg ur_type)"
@@ -24,4 +31,3 @@
         <origin xyz="0 0 0" rpy="0 0 0" />
     </xacro:ur_robot>
-    <xacro:workcell_ros2_control name="WebotsControl" initial_positions_file="$(arg initial_positions_file)"/>
 </robot>
