Commit message: update workcell_webots to run on jazzy, sim is running, but without use_sim_time: True

File: workcell/workcell_webots/config/ur5e_webots.urdf.xacro (robot description, xacro)
@@ -2,5 +2,5 @@
 <robot name="ur5e" xmlns:xacro="http://www.ros.org/wiki/xacro">
     <!-- Args -->
-    <xacro:arg name="initial_positions_file" default="initial_positions.yaml" />
+    <xacro:arg name="initial_positions_file" default="$(find workcell_moveit_config)/config/initial_positions.yaml"/>
     <xacro:arg name="ur_type" default="ur5e"/>
     <xacro:arg name="joint_limits_parameters_file" default="$(find ur_description)/config/$(arg ur_type)/joint_limits.yaml"/>
@@ -28,6 +28,6 @@
         physical_parameters_file="$(arg physical_parameters_file)"
         visual_parameters_file="$(arg visual_parameters_file)"
-        generate_ros2_control_tag="false">
-        <origin xyz="0 0 0" rpy="0 0 0" />
+        >
+        <origin xyz="0 0 0" rpy="0 0 0"/>
     </xacro:ur_robot>
 </robot>
