Commit message: update workcell_control to work on jazzy (from humble)

File: workcell/workcell_control/urdf/workcell_controlled.urdf.xacro (robot description, xacro)
@@ -4,5 +4,5 @@
   <xacro:include filename="$(find workcell_description)/urdf/workcell_macro.xacro"/>
   <!--The driver already provides a control tag for the UR arm, we can directly include-->
-  <xacro:include filename="$(find ur_description)/urdf/ur.ros2_control.xacro"/>
+  <xacro:include filename="$(find ur_robot_driver)/urdf/ur.ros2_control.xacro"/>
   <!--We need to specify the arguments used for parametrizing our description-->
   <xacro:arg name="ur_type" default="ur5e"/>
@@ -20,9 +20,6 @@
   <xacro:arg name="ur_output_recipe_filename" default="$(find ur_robot_driver)/resources/rtde_output_recipe.txt"/>
   <xacro:arg name="ur_input_recipe_filename" default="$(find ur_robot_driver)/resources/rtde_input_recipe.txt"/>
-  <xacro:arg name="use_fake_hardware" default="false" />
-  <xacro:arg name="fake_sensor_commands" default="false" />
-  <!--find hash_kinematics in kinematics_params-->
-  <xacro:property name="kinematics_params_file" value="$(arg kinematics_params)"/>
-  <xacro:property name="kinematics_hash" value="${xacro.load_yaml(kinematics_params_file)['kinematics']['hash']}"/>
+  <xacro:arg name="use_mock_hardware" default="false" />
+  <xacro:arg name="mock_sensor_commands" default="false" />
   <!-- World Link (represents the origin of the world coordinate frame) -->
   <link name="world"/>
@@ -45,13 +42,12 @@
     name="$(arg ur_type)"
     tf_prefix="$(arg ur_type)_"
-    hash_kinematics="${kinematics_hash}"
+    kinematics_parameters_file="$(arg kinematics_parameters_file)"
     robot_ip="$(arg robot_ip)"
     script_filename="$(arg ur_script_filename)"
     output_recipe_filename="$(arg ur_output_recipe_filename)"
     input_recipe_filename="$(arg ur_input_recipe_filename)"
-    use_fake_hardware="$(arg use_fake_hardware)"
-    fake_sensor_commands="$(arg fake_sensor_commands)"
+    use_mock_hardware="$(arg use_mock_hardware)"
+    mock_sensor_commands="$(arg mock_sensor_commands)"
     headless_mode="$(arg headless_mode)"
   />
-  <!--If you had more controlled devices in your description, e.g. a gripper, you can add another ros2_control tag here-->
 </robot>
